File: circuit/FrugalWatchdog.sch (KiCad schematic (older format))
At the start: 5 parts

Commit message: Update the schematic and firmware to match reality.
Connections:
- net at IC?.4 (GND), P?.1 (P1), R?.2: no longer IC?.1 (PB5(~RESET~/dW/ADC0/PCINT5))
- net at IC?.8 (VCC), P?.4 (P4), P?.5 (P5): now also IC?.1 (PB5(~RESET~/dW/ADC0/PCINT5))
Changed lines of the file:
@@
 GND
 Text Notes 3050 3700 0    60   ~ 0
+TXD
+Text Notes 3050 3600 0    60   ~ 0
 RXD
-Text Notes 3050 3600 0    60   ~ 0
-TXD
 Text Notes 3050 3500 0    60   ~ 0
 3V3
@@
 Wire Wire Line
 	3550 3600 3050 3600
-Wire Wire Line
-	4050 3700 4050 4100
 Wire Wire Line
 	3600 3300 4050 3300
@@
 Wire Wire Line
 	3600 4100 6750 4100
-Connection ~ 4050 4100
 Wire Wire Line
 	3900 3600 4050 3600
@@
 Wire Wire Line
 	3600 3700 3600 3300
+Wire Wire Line
+	4050 3700 3650 3700
+Wire Wire Line
+	3650 3700 3650 2950
+Connection ~ 3650 2950
 $EndSCHEMATC
